File: pcb/home_checker/home_mon.kicad_pcb (KiCad board)
At the start: 2 copper layers, 102.9 x 81.6 mm, 16 parts, among them J12 220va, J14 J14, J15 J13, J4 J15, J5 J16, J6 UART, J7 Jumper, J8 T° sensor, J9 Alim, K1 FINDER-40.52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

Commit message: feat: Monitor the battery voltage
Parts:
- added J1: V Bat, TestPoint:TestPoint_Loop_D1.80mm_Drill1.0mm_Beaded, F.Cu at (66.4, 86.5)
- added R4: 100k, Resistor_THT:R_Axial_DIN0207_L6.3mm_D2.5mm_P10.16mm_Horizontal, F.Cu at (69.9, 93.9)
- added R5: 33k, Resistor_THT:R_Axial_DIN0207_L6.3mm_D2.5mm_P10.16mm_Horizontal, F.Cu at (73.2, 83.7)
- moved R3 3.54 mm to (72.5, 100.5)
- moved J15 2.03 mm to (159.1, 118.0)
- moved J5 2.03 mm to (111.1, 134.5)
- moved J4 2.03 mm to (111.1, 112.9)
- moved J6 2.03 mm to (113.6, 67.2)
- moved J14 2.03 mm to (159.1, 135.8)
- moved J7 0.76 mm to (65.6, 95.6)
Connections:
- U1 pad 3: unconnected-(U1-GPIO39-Pad3) -> Bat
Routing:
- net Bat: track 0.00 -> 9.21 mm
- net GND: track 464.6 -> 471.0 mm
- net +5V: track 235.6 -> 229.8 mm
- net Net-(J1-Pin_1): track 0.00 -> 5.75 mm
- net Net-(J4-Pin_2): track 21.6 -> 23.8 mm
- net Net-(J6-Pin_4): track 60.3 -> 62.0 mm
- net Net-(J6-Pin_3): track 69.9 -> 71.5 mm
- net Net-(J7-Pin_3): track 16.5 -> 15.1 mm
- net Net-(J7-Pin_2): track 35.5 -> 36.4 mm
- net Net-(J7-Pin_1): track 13.0 -> 13.6 mm
Other:
- board text added: "Home Check V1.1"
- board text removed: "Home Check V1.0"

Commit message: fix: Make the sending of sending operational again (canary exception) Make the ADC more reliable
Parts:
- R4: value 100k -> 10k
- R5: value 33k -> 2,7k
Changed lines of the file:
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@@
 			)
 		)
-		(property "Value" "33k"
+		(property "Value" "2,7k"
 			(at 4.9908 -1.524 90)
 			(layer "F.Fab")
@@
 			)
 		)
-		(property "Value" "100k"
+		(property "Value" "10k"
 			(at 5.08 1.37 90)
 			(layer "F.Fab")
